Commit message: Add simple navigation package and simple arduino diff drive

File: non_ws/src/robokrub-base-v3_description/urdf/_d435.gazebo.xacro (robot description, xacro)
@@ -131,5 +131,5 @@
       	<rangeMinDepth>0.2</rangeMinDepth>
       	<rangeMaxDepth>10.0</rangeMaxDepth>
-      	<pointCloud>false</pointCloud>
+      	<pointCloud>true</pointCloud>
       	<pointCloudTopicName>depth/points</pointCloudTopicName>
       	<pointCloudCutoff>0.5</pointCloudCutoff>

File: non_ws/src/robokrub-base-v3_description/urdf/robokrub-base-v3.xacro (robot description, xacro)
@@ -8,9 +8,9 @@
     <parent link="base_footprint"/>
     <child link="base_link"/>
-    <origin xyz="0.0 0.0 0.010" rpy="0 0 0"/>
+    <origin xyz="0.0 0.0 0.010" rpy="0 0 3.14"/>
   </joint>
   <link name="base_link">
     <inertial>
-      <origin rpy="0 0 3.14" xyz="0.12439966211944935 -0.00012861812803782383 0.016903695260053322"/>
+      <origin rpy="0 0 -3.14" xyz="0.12439966211944935 -0.00012861812803782383 0.016903695260053322"/>
       <mass value="27.36387050855292"/>
       <inertia ixx="0.608767" ixy="-0.000793" ixz="0.05113" iyy="0.461089" iyz="-6.3e-05" izz="0.865635"/>
@@ -32,5 +32,5 @@
   <link name="Lidar_v2_1">
     <inertial>
-      <origin rpy="0 0 0" xyz="-0.13151592549315028 0.0005322844293224717 0.024735037477504607"/>
+      <origin rpy="0 0 -3.14" xyz="-0.13151592549315028 0.0005322844293224717 0.024735037477504607"/>
       <mass value="0.07746853107841598"/>
       <inertia ixx="3.4e-05" ixy="-1e-06" ixz="-7e-06" iyy="6.5e-05" iyz="-0.0" izz="7.6e-05"/>
@@ -186,5 +186,5 @@
   <xacro:include filename="$(find robokrub-base-v3_description)/urdf/_d435.urdf.xacro" />
   <xacro:sensor_d435 name="sensor_d435" parent="base_link">
-    <origin xyz="-0.0525 0.0 0.3" rpy="0 0 -3.14"/>
+    <origin xyz="-0.0525 0.0 0.3" rpy="0 0 3.14"/>
     <!-- <origin xyz="0 0 0" rpy="${-90.0 * deg_to_rad} 0 ${-90.0 * deg_to_rad}"/> -->
   </xacro:sensor_d435>
